Commit message: Create a Gazebo Robot Model demo with repair Gazebo can't start.

File: gazebo_env/robot_biped.urdf (robot description, URDF)
Before this commit: robot humanoid_biped, 6 links, 5 joints
Links:
- removed link left_leg_link
- removed link right_leg_link
- added link left_arm_link, mass 1.0; collision cylinder length=0.2 radius=0.05; visual cylinder length=0.2 radius=0.05
- added link left_foot_link, mass 0.8; collision box size=0.15 0.1 0.05; visual box size=0.15 0.1 0.05
- added link left_shin_link, mass 1.5; collision cylinder length=0.225 radius=0.08; visual cylinder length=0.225 radius=0.08
- added link left_thigh_link, mass 1.5; collision cylinder length=0.225 radius=0.08; visual cylinder length=0.225 radius=0.08
- added link right_arm_link, mass 1.0; collision cylinder length=0.2 radius=0.05; visual cylinder length=0.2 radius=0.05
- added link right_foot_link, mass 0.8; collision box size=0.15 0.1 0.05; visual box size=0.15 0.1 0.05
- added link right_shin_link, mass 1.5; collision cylinder length=0.225 radius=0.08; visual cylinder length=0.225 radius=0.08
- added link right_thigh_link, mass 1.5; collision cylinder length=0.225 radius=0.08; visual cylinder length=0.225 radius=0.08
- link left_camera_link: mass 0.08 -> 0.01; geometry collision box size=0.02 0.02 0.02; visual box size=0.02 0.02 0.02
- link right_camera_link: mass 0.08 -> 0.01; geometry collision box size=0.02 0.02 0.02; visual box size=0.02 0.02 0.02
Joints:
- removed joint left_leg_joint
- removed joint right_leg_joint
- added joint left_ankle_joint: type revolute, parent left_shin_link, child left_foot_link, origin xyz=0 0 -0.225 rpy=0 0 0, axis 0 1 0, limit lower=-0.5 upper=0.5 effort=50 velocity=2.0
- added joint left_hip_joint: type revolute, parent base_link, child left_thigh_link, origin xyz=0 0.12 -0.275 rpy=0 0 0, axis 0 0 1, limit lower=-1.57 upper=1.57 effort=100 velocity=3.0
- added joint left_knee_joint: type revolute, parent left_thigh_link, child left_shin_link, origin xyz=0 0 -0.225 rpy=0 0 0, axis 0 0 1, limit lower=0 upper=1.57 effort=100 velocity=3.0
- added joint left_shoulder_joint: type revolute, parent base_link, child left_arm_link, origin xyz=0.1 0.15 0.1 rpy=0 0 0, axis 0 0 1, limit lower=-1.57 upper=1.57 effort=50 velocity=2.0
- added joint right_ankle_joint: type revolute, parent right_shin_link, child right_foot_link, origin xyz=0 0 -0.225 rpy=0 0 0, axis 0 1 0, limit lower=-0.5 upper=0.5 effort=50 velocity=2.0
- added joint right_hip_joint: type revolute, parent base_link, child right_thigh_link, origin xyz=0 -0.12 -0.275 rpy=0 0 0, axis 0 0 1, limit lower=-1.57 upper=1.57 effort=100 velocity=3.0
- added joint right_knee_joint: type revolute, parent right_thigh_link, child right_shin_link, origin xyz=0 0 -0.225 rpy=0 0 0, axis 0 0 1, limit lower=0 upper=1.57 effort=100 velocity=3.0
- added joint right_shoulder_joint: type revolute, parent base_link, child right_arm_link, origin xyz=0.1 -0.15 0.1 rpy=0 0 0, axis 0 0 1, limit lower=-1.57 upper=1.57 effort=50 velocity=2.0
- joint head_joint: axis (none) -> 0 1 0; limit (none) -> lower=-0.5 upper=0.5 effort=20 velocity=1.0; origin xyz=0 0 0.4 rpy=0 0 0 -> xyz=0 0 0.275 rpy=0 0 0; type fixed -> revolute
- joint left_camera_joint: origin xyz=0.04 0.08 0 rpy=0 0 0 -> xyz=0.06 0.08 0 rpy=0 0 0
- joint right_camera_joint: origin xyz=0.04 -0.08 0 rpy=0 0 0 -> xyz=0.06 -0.08 0 rpy=0 0 0
